File: electronics/tesla-seat-controller-shield/tesla-seat-controller-shield.kicad_pcb (KiCad board)
At the start: 2 copper layers, 68.8 x 53.6 mm, 12 parts, among them J1 12V In, J2 Motor Driver, J3 Fan Upper, J4 Fan Lower, J5 Switchpack

Commit message: Update part positions and remove 12v Vin
Parts:
- moved J4 0.90 mm to (104.9, 80.0)
- moved J2 0.38 mm to (106.8, 91.7)
Connections:
- A1 pad 8: +12V -> unconnected-(A1-VIN-Pad8)
Routing:
- net +12V: track 103.0 -> 70.1 mm
- net GND: vias 2 -> 3
