File: electronics/tesla-seat-controller-shield/tesla-seat-controller-shield.kicad_sch (KiCad schematic)
At the start: 12 parts, among them J1 12V In, J2 Motor Driver, J3 Fan Upper, J4 Fan Lower, J5 Switchpack

Commit message: Mirror Arduino shield and update some documentation paths
Connections:
- net switch_backrest_track: now also J5.4 (Pin_4); no longer J5.2 (Pin_2)
- net switch_lumbar: now also J5.2 (Pin_2); no longer J5.4 (Pin_4)
Other:
- moved on the sheet: J5
Changed lines of the file:
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@@
 	(wire
 		(pts
-			(xy 233.68 76.2) (xy 233.68 88.9)
+			(xy 233.68 86.36) (xy 233.68 88.9)
 		)
 		(stroke
@@
 	(wire
 		(pts
-			(xy 234.95 76.2) (xy 233.68 76.2)
-		)
-		(stroke
-			(width 0)
-			(type default)
-		)
-	)
-	(wire
-		(pts
 			(xy 58.42 60.96) (xy 69.85 60.96)
 		)
@@
 		(pts
 			(xy 76.2 55.88) (xy 76.2 71.12)
+		)
+		(stroke
+			(width 0)
+			(type default)
+		)
+	)
+	(wire
+		(pts
+			(xy 233.68 86.36) (xy 234.95 86.36)
 		)
 		(stroke
@@
 	(symbol
 		(lib_id "Connector:Conn_01x04_Pin")
-		(at 240.03 78.74 0)
-		(mirror y)
+		(at 240.03 83.82 180)
 		(unit 1)
 		(exclude_from_sim no)
@@
 		(dnp no)
 		(property "Reference" "J5"
-			(at 241.3 78.7399 0)
+			(at 241.3 83.8201 0)
 			(effects
 				(font
@@
 		)
 		(property "Value" "Switchpack"
-			(at 241.3 81.2799 0)
+			(at 241.3 81.2801 0)
 			(effects
 				(font
@@
 		)
 		(property "Footprint" "Connector_PinHeader_2.54mm:PinHeader_1x04_P2.54mm_Vertical"
-			(at 240.03 78.74 0)
+			(at 240.03 83.82 0)
 			(effects
 				(font
@@
 		)
 		(property "Datasheet" "~"
-			(at 240.03 78.74 0)
+			(at 240.03 83.82 0)
 			(effects
 				(font
@@
 		)
 		(property "Description" "Generic connector, single row, 01x04, script generated"
-			(at 240.03 78.74 0)
-			(effects
-				(font
+			(at 240.03 83.82 0)
+			(effects
+				(font

Commit message: Add 3D models and make board updates to match shield layout
Connections:
- net +12V: now also J2.1 (Pin_1); no longer J2.2 (Pin_2)
- net GND: now also J2.2 (Pin_2); no longer J2.1 (Pin_1)
Changed lines of the file:
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@@
 	(symbol
 		(lib_id "Connector:Screw_Terminal_01x02")
-		(at 85.09 120.65 0)
-		(mirror x)
+		(at 85.09 118.11 0)
 		(unit 1)
 		(exclude_from_sim no)
@@
 		(dnp no)
 		(property "Reference" "J2"
-			(at 87.63 120.6501 0)
+			(at 87.63 118.1099 0)
 			(effects
 				(font
@@
 		)
 		(property "Value" "Motor Driver"
-			(at 87.63 118.1101 0)
+			(at 87.63 120.6499 0)
 			(effects
 				(font
@@
 		)
 		(property "Footprint" "TerminalBlock:TerminalBlock_bornier-2_P5.08mm"
-			(at 85.09 120.65 0)
+			(at 85.09 118.11 0)
 			(effects
 				(font
@@
 		)
 		(property "Datasheet" "~"
-			(at 85.09 120.65 0)
+			(at 85.09 118.11 0)
 			(effects
 				(font
@@
 		)
 		(property "Description" "Generic screw terminal, single row, 01x02, script generated (kicad-library-utils/schlib/autogen/connector/)"
-			(at 85.09 120.65 0)
+			(at 85.09 118.11 0)
 			(effects
 				(font

Commit message: Update part positions and remove 12v Vin
Connections:
- net +12V: no longer A1.8 (VIN)
- no-connect marks 23 -> 24
Changed lines of the file:
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@@
+	)
+	(no_connect
+		(at 132.08 48.26)
 	)
 	(no_connect
@@
 		(pts
 			(xy 76.2 50.8) (xy 76.2 55.88)
-		)
-		(stroke
-			(width 0)
-			(type default)
-		)
-	)
-	(wire
-		(pts
-			(xy 132.08 41.91) (xy 132.08 48.26)
 		)
 		(stroke
@@
 					(unit 1)
 				)
-			)
-		)
-	)
-	(symbol
-		(lib_id "power:+12V")
-		(at 132.08 41.91 0)
-		(unit 1)
-		(exclude_from_sim no)
-		(in_bom yes)
-		(on_board yes)
-		(dnp no)
-		(fields_autoplaced yes)
-		(property "Reference" "#PWR03"
-			(at 132.08 45.72 0)
-			(effects
-				(font
-					(size 1.27 1.27)
-				)
-				(hide yes)
-			)
-		)
-		(property "Value" "+12V"
-			(at 132.08 36.83 0)
-			(effects
-				(font
-					(size 1.27 1.27)
-				)
-			)
-		)
-		(property "Footprint" ""
-			(at 132.08 41.91 0)
-			(effects
-				(font
-					(size 1.27 1.27)
-				)
-				(hide yes)
-			)
-		)
-		(property "Datasheet" ""
-			(at 132.08 41.91 0)
-			(effects
-				(font
-					(size 1.27 1.27)
-				)
-				(hide yes)
-			)
-		)
-		(property "Description" "Power symbol creates a global label with name \"+12V\""
-			(at 132.08 41.91 0)
-			(effects
-				(font
-					(size 1.27 1.27)
-				)
-				(hide yes)
-			)
-		)
-		(pin "1"
-		)
-		(instances
-			(project ""
-				(path "/24f488f1-5e6b-4fe6-984e-19086c29a5ad"
-					(reference "#PWR03")
-					(unit 1)
-				)

Commit message: Reshuffle pins
Connections:
- net fan_lower_pwm: now also A1.26 (D11); no longer A1.21 (D6)
- net fan_upper_pwm: now also A1.24 (D9); no longer A1.20 (D5)
- net motor_s1_m1_dir: now reaches A1.17 (D2)
- net motor_s1_m1_pwm: now reaches A1.18 (D3)
- net motor_s2_m1_dir: now reaches A1.19 (D4)
- net motor_s1_m2_dir: now reaches A1.22 (D7)
- net motor_s2_m2_pwm: now reaches A1.25 (D10)
- net motor_s2_m2_dir: now reaches A1.27 (D12)
- new net motor_s1_m2_pwm: A1.21 (D6)
- new net motor_s2_m1_pwm: A1.20 (D5)
Other:
- moved on the sheet: J3, J4
