File: electronics/tesla-seat-controller/tesla-seat-controller.kicad_sch (KiCad schematic)
At the start: 37 parts, among them J1 USB_C_Receptacle, J2 SWD, J3 12V In, SW1 SW_Push, U1 RP2354, U2 AP63203WU, Y1 ABM8-272-T3

Commit message: Add standalone seat-controller schematic: RP2354 + dual DRV8262 drivers
Build out the non-shield board around an RP2354B with two DRV8262
dual-H-bridge motor drivers (4 seat motors total), using one reusable
motor-driver hierarchical sheet instanced twice.

- motor-driver.kicad_sch: DRV8262 in dual-H-bridge PWM mode (MODE1=GND,
  MODE2=DVDD), charge pump, VREF divider (~3.3V), IPROPI sense (3.09k,
  ~5A trip), per-motor 2-pin output connectors. Verified via netlist.
- Root: RP2354B core regulator (3.3uH + 4.7uF, 33ohm/4.7uF AVDD filter),
  12MHz crystal, USB-C, SWD, BOOTSEL, AP63203 3.3V buck, RUN reset RC.
  Values cross-checked against the RP2350 hardware design guide.
- Clean up the SnapEDA DRV8262 symbol: rename mode-multiplexed slash
  pins to DDW dual-mode names, retype OUT/VREF pins to passive.
- ERC clean (0 violations).

Known TODO before fab: nFAULT pull-ups added; still need fan drivers,
12V input bulk + reverse-polarity/fuse protection, VM cap voltage
ratings, ADC_AVDD filter.

Co-Authored-By: Claude Opus 4.8 <noreply@anthropic.com>
Parts:
- added C37: 100nF, symbol Device:C_Small
- added R15, R16: 1k, symbol Device:R_Small
- R3: renamed from R5; value 27R -> 27
- R4: renamed from R6; value 27R -> 27
- R6: renamed from R4; value 33R -> 33
- renumbered C20 to C11, C11 to C12, C21 to C13, C12 to C14, C22 to C15, C13 to C16, C14 to C17, C15 to C18, C16 to C19, C5 to C2, C17 to C20, C18 to C21, C19 to C22, C6 to C3, C3 to C4, C4 to C5, C2 to C6, C9 to C7, C7 to C9, J3 to J1, J1 to J3, R2 to R1, R1 to R2, R3 to R5, U2 to U1, U1 to U2
Connections:
- net IOVDD is gone; now on net +3V3: U2.15 (IOVDD), U2.24 (IOVDD), U2.29 (IOVDD), U2.41 (IOVDD), U2.5 (IOVDD), U2.50 (IOVDD), U2.59 (ADC_AVDD), U2.60 (IOVDD), U2.68 (USB_OTP_VDD), U2.69 (QSPI_IOVDD), U2.76 (IOVDD)
- net +3V3: now also R15.1
- net GND: now also J3.SH (SHIELD), C37.1; no longer J3.S1 (SHIELD)
- net at SW1.1: now also R16.1; no longer U2.75 (~{QSPI_SS})
- net Motor Driver CD/A_IN1: now reaches U2.1 (GPIO4)
- net Motor Driver CD/A_IN2: now reaches U2.2 (GPIO5)
- net Motor Driver CD/B_IN1: now reaches U2.3 (GPIO6)
- net at U2.35 (RUN): now also C37.2, R15.2
- net Motor Driver CD/B_IN2: now reaches U2.4 (GPIO7)
- net A_ISNS: now reaches U2.49 (GPIO40/ADC0)
- net B_ISNS: now reaches U2.52 (GPIO41/ADC1)
- net C_ISNS: now reaches U2.53 (GPIO42/ADC2)
- net D_ISNS: now reaches U2.54 (GPIO43/ADC3)
- net ~{AB_SLEEP}: now reaches U2.6 (GPIO8)
- net ~{AB_FAULT}: now reaches U2.7 (GPIO9)
- net Motor Driver AB/A_IN1: now reaches U2.77 (GPIO0)
- net Motor Driver AB/A_IN2: now reaches U2.78 (GPIO1)
- net Motor Driver AB/B_IN1: now reaches U2.79 (GPIO2)
- net ~{CD_SLEEP}: now reaches U2.8 (GPIO10)
- net Motor Driver AB/B_IN2: now reaches U2.80 (GPIO3)
- net ~{CD_FAULT}: now reaches U2.9 (GPIO11)
- new net: R16.2, U2.75 (~{QSPI_SS})
- no-connect marks 6 -> 37
Other:
- added sheet Motor Driver AB (motor-driver.kicad_sch)
- added sheet Motor Driver CD (motor-driver.kicad_sch)
- moved on the sheet: C2, C3, C7, C8, C9, L2, R3, R4, R5, R6, SW1, U2
