File: electronics/tesla-seat-controller/tesla-seat-controller.kicad_sch (KiCad schematic)
At the start: 52 parts, among them J1 12V IN, J2 SWD, J3 USB-C, J8 Fan A, J9 Fan B, Q1 IPD90P03P4L-04, Q2 2N7002, Q3 2N7002, SW1 SW_Push, U1 AP63203WU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

Commit message: wip
Parts:
- removed C7, C8, C9: 4.7uF, symbol Device:C_Small
- removed L2: 3.3uH, symbol Device:L_Small
- removed R6: 33, symbol Device:R_Small
- removed U2: RP2354, Package_DFN_QFN:QFN-80-1EP_10x10mm_P0.4mm_EP3.4x3.4mm, symbol MCU_RaspberryPi:RP2354B
- added U2: STM32G0B1CBTx, Package_QFP:LQFP-48_7x7mm_P0.5mm, symbol MCU_ST_STM32G0:STM32G0B1CBTx
Connections:
- net GND: now also U2.7 (VSS)
- no-connect marks 36 -> 6
