File: electronics/tesla-seat-controller/tesla-seat-controller.kicad_sch (KiCad schematic)
At the start: 37 parts, among them J1 12V IN, J2 Fan A, J3 Fan B, J4 TC2030, J5 Switchpack, Q1 IPD90P03P4L-04, Q2 2N7002, Q3 2N7002, U1 STM32G0B1CBTx, U2 AP63203WU

Commit message: Complete PCB layout: 4-layer, GND/GNDPWR split, 3D models, DRC clean
- 4-layer stackup: In1 split ground planes (GND logic / GNDPWR power,
  joined by net tie NT1 at J1), In2 partial +12V plane
- Schematic: GNDPWR net for motor/power return paths (PGND pins, VM
  bypass + bulk caps, battery return, TVS, fans); logic/analog stays
  on GND (IPROPI sense, VREF, DVDD, MCU, buck)
- Both DRV8262 channels placed and routed (multichannel clone), solid
  pad connections on all power zones, per-cluster VM bypass
- 3D models: XT30PW-M/F (LCSC) and DRV8262 DDW stand-in restored from
  history, aligned transforms; drop custom symbol lib and fp-lib-table
  in favor of official libraries
- Net classes Power/Motor (visual grouping only)
- DRC: 0 violations, 0 unconnected
Parts:
- added NT1: NetTie_2, symbol Device:NetTie_2
- R2: value 100k -> 10k
Connections:
- net GND: now also NT1.2; no longer D2.2 (A), J1.1 (Pin_1), J2.3 (Pin_3), J3.3 (Pin_3), Q2.2 (S), Q3.2 (S), R2.2
- new net GNDPWR: D2.2 (A), J1.1 (Pin_1), J2.3 (Pin_3), J3.3 (Pin_3), NT1.1, Q2.2 (S), Q3.2 (S), R2.2
