File: electronics/tesla-seat-controller/motor-driver.kicad_sch (KiCad schematic)
At the start: 15 parts, among them J6 Motor A, J7 Motor B, U3 DRV8262DDVR

Commit message: Complete PCB layout: 4-layer, GND/GNDPWR split, 3D models, DRC clean
- 4-layer stackup: In1 split ground planes (GND logic / GNDPWR power,
  joined by net tie NT1 at J1), In2 partial +12V plane
- Schematic: GNDPWR net for motor/power return paths (PGND pins, VM
  bypass + bulk caps, battery return, TVS, fans); logic/analog stays
  on GND (IPROPI sense, VREF, DVDD, MCU, buck)
- Both DRV8262 channels placed and routed (multichannel clone), solid
  pad connections on all power zones, per-cluster VM bypass
- 3D models: XT30PW-M/F (LCSC) and DRV8262 DDW stand-in restored from
  history, aligned transforms; drop custom symbol lib and fp-lib-table
  in favor of official libraries
- Net classes Power/Motor (visual grouping only)
- DRC: 0 violations, 0 unconnected
Parts:
- added C27, C29: 1nF, Capacitor_SMD:C_0805_2012Metric, symbol Device:C_Small
- J8: renamed from J7; value Motor B -> Motor A
- J9: renamed from J6; value Motor A -> Motor B
- U3: footprint tesla-seat-controller:HTSSOP44-DDV_TEX -> Package_SO:HTSSOP-44_6.1x14mm_P0.635mm_TopEP4.14x7.01mm
Connections:
- net A_IN1: now also U3.28 (IN3); no longer U3.26 (IN1)
- net A_IN2: now also U3.29 (IN4); no longer U3.27 (IN2)
- net A_ISNS: now also R8.2, U3.37 (IPROPI2), C27.2; no longer R9.2, U3.36 (IPROPI1)
- net B_IN1: now also U3.26 (IN1); no longer U3.28 (IN3)
- net B_IN2: now also U3.27 (IN2); no longer U3.29 (IN4)
- net B_ISNS: now also R9.2, U3.36 (IPROPI1), C29.2; no longer R8.2, U3.37 (IPROPI2)
- net GND: now also C27.1, C29.1; no longer C17.2, C18.2, C19.2, U3.10 (PGND34), U3.13 (PGND12), U3.20 (PGND12), U3.3 (PGND34)
- net AOUT2: now reaches U3.4 (OUT3), U3.5 (OUT3), U3.6 (OUT3)
- net AOUT2: now also J8.2 (Pin_2); no longer J8.1 (Pin_1)
- net AOUT1: now reaches U3.7 (OUT4), U3.8 (OUT4), U3.9 (OUT4)
- net AOUT1: now also J8.1 (Pin_1); no longer J8.2 (Pin_2)
- net BOUT1: now reaches J9.1 (Pin_1), U3.17 (OUT1), U3.18 (OUT1), U3.19 (OUT1)
- net BOUT2: now reaches J9.2 (Pin_2), U3.14 (OUT2), U3.15 (OUT2), U3.16 (OUT2)
- new net GNDPWR: C17.2, C18.2, C19.2, U3.10 (PGND34), U3.13 (PGND12), U3.20 (PGND12), U3.3 (PGND34)
Other:
- moved on the sheet: J8, J9, R8, R9
