File: electronics/tesla-seat-controller/tesla-seat-controller.kicad_pcb (KiCad board)
At the start: 0 parts

Commit message: Complete PCB layout: 4-layer, GND/GNDPWR split, 3D models, DRC clean
- 4-layer stackup: In1 split ground planes (GND logic / GNDPWR power,
  joined by net tie NT1 at J1), In2 partial +12V plane
- Schematic: GNDPWR net for motor/power return paths (PGND pins, VM
  bypass + bulk caps, battery return, TVS, fans); logic/analog stays
  on GND (IPROPI sense, VREF, DVDD, MCU, buck)
- Both DRV8262 channels placed and routed (multichannel clone), solid
  pad connections on all power zones, per-cluster VM bypass
- 3D models: XT30PW-M/F (LCSC) and DRV8262 DDW stand-in restored from
  history, aligned transforms; drop custom symbol lib and fp-lib-table
  in favor of official libraries
- Net classes Power/Motor (visual grouping only)
- DRC: 0 violations, 0 unconnected
Parts:
- added C1: 100nF, Capacitor_SMD:C_0805_2012Metric, F.Cu at (170.9, 67.2)
- added C10: 100nF, Capacitor_SMD:C_0805_2012Metric, F.Cu at (174.7, 62.0)
- added C11: 100nF, Capacitor_SMD:C_0805_2012Metric, F.Cu at (175.2, 64.8)
- added C12: 4.7uF, Capacitor_SMD:C_0805_2012Metric, F.Cu at (174.7, 60.0)
- added C13: 100nF, Capacitor_SMD:C_0805_2012Metric, F.Cu at (178.6, 81.8)
- added C14: 1uF, Capacitor_SMD:C_0805_2012Metric, F.Cu at (167.1, 77.0)
- added C15: 100nF, Capacitor_SMD:C_0805_2012Metric, F.Cu at (164.1, 77.0)
- added C16: 1uF, Capacitor_SMD:C_0805_2012Metric, F.Cu at (179.6, 88.3)
- added C17: 220uF 35V polymer, Capacitor_SMD:CP_Elec_10x10.5, F.Cu at (155.9, 80.0)
- added C18: 10nF, Capacitor_SMD:C_0805_2012Metric, F.Cu at (161.0, 89.0)
- added C19: 10nF, Capacitor_SMD:C_0805_2012Metric, F.Cu at (179.1, 90.7)
- added C2: 100nF, Capacitor_SMD:C_0805_2012Metric, F.Cu at (210.2, 73.0)
- added C20: 100nF, Capacitor_SMD:C_0805_2012Metric, F.Cu at (210.6, 81.8)
- added C21: 1uF, Capacitor_SMD:C_0805_2012Metric, F.Cu at (199.1, 77.0)
- added C22: 100nF, Capacitor_SMD:C_0805_2012Metric, F.Cu at (196.1, 77.0)
- added C23: 1uF, Capacitor_SMD:C_0805_2012Metric, F.Cu at (211.6, 88.3)
- added C24: 220uF 35V polymer, Capacitor_SMD:CP_Elec_10x10.5, F.Cu at (187.9, 80.0)
- added C25: 10nF, Capacitor_SMD:C_0805_2012Metric, F.Cu at (193.0, 88.9)
- added C26: 10nF, Capacitor_SMD:C_0805_2012Metric, F.Cu at (211.1, 90.7)
- added C27: 1nF, Capacitor_SMD:C_0805_2012Metric, F.Cu at (174.6, 69.4)
- added C28: 1nF, Capacitor_SMD:C_0805_2012Metric, F.Cu at (178.7, 71.5)
- added C29: 1nF, Capacitor_SMD:C_0805_2012Metric, F.Cu at (175.3, 73.4)
- added C3: 10uF, Capacitor_SMD:C_1206_3216Metric, F.Cu at (165.6, 66.3)
- added C30: 1nF, Capacitor_SMD:C_0805_2012Metric, F.Cu at (180.7, 71.5)
- added C4: 22uF, Capacitor_SMD:C_1206_3216Metric, F.Cu at (160.3, 56.9)
- added C5: 22uF, Capacitor_SMD:C_1206_3216Metric, F.Cu at (160.3, 59.4)
- added C6: 100nF, Capacitor_SMD:C_0805_2012Metric, F.Cu at (168.9, 63.2)
- added C7: 100nF, Capacitor_SMD:C_0805_2012Metric, F.Cu at (137.0, 65.0)
- added C8: 100nF, Capacitor_SMD:C_0805_2012Metric, F.Cu at (137.0, 67.5)
- added C9: 100nF, Capacitor_SMD:C_0805_2012Metric, F.Cu at (137.0, 70.0)
- added D1: BZT52C12, Diode_SMD:D_SOD-123, F.Cu at (213.2, 73.5)
- added D2: SMBJ16A, Diode_SMD:D_SMB, F.Cu at (204.0, 66.8)
- added F1: 10A (mini blade), Fuse:Fuseholder_Blade_Mini_Keystone_3568, F.Cu at (203.0, 60.5)
- added J1: 12V IN, Connector_AMASS:AMASS_XT30PW-M_1x02_P2.50mm_Horizontal, F.Cu at (209.0, 66.0)
- added J2: Fan A, Connector_JST:JST_XH_S3B-XH-A_1x03_P2.50mm_Horizontal, F.Cu at (131.9, 82.8)
- added J3: Fan B, Connector_JST:JST_XH_S3B-XH-A_1x03_P2.50mm_Horizontal, F.Cu at (131.9, 95.5)
- added J4: TC2030, Connector:Tag-Connect_TC2030-IDC-NL_2x03_P1.27mm_Vertical, F.Cu at (185.0, 55.5)
- added J5: Switchpack, Connector_JST:JST_XH_S4B-XH-A_1x04_P2.50mm_Horizontal, F.Cu at (132.0, 62.5)
- added J6: Motor A, Connector_AMASS:AMASS_XT30PW-F_1x02_P2.50mm_Horizontal, F.Cu at (196.5, 96.8)
- added J7: Motor B, Connector_AMASS:AMASS_XT30PW-F_1x02_P2.50mm_Horizontal, F.Cu at (212.5, 96.8)
- added J8: Motor A, Connector_AMASS:AMASS_XT30PW-F_1x02_P2.50mm_Horizontal, F.Cu at (164.5, 96.8)
- added J9: Motor B, Connector_AMASS:AMASS_XT30PW-F_1x02_P2.50mm_Horizontal, F.Cu at (180.5, 96.8)
- added L1: 3.9uH, Inductor_SMD:L_Bourns_SRN6045TA, F.Cu at (166.9, 58.2)
- added Q1: IPD90P03P4L-04, Package_TO_SOT_SMD:TO-252-2, F.Cu at (194.6, 66.9)
- added Q2: 2N7002, Package_TO_SOT_SMD:SOT-23, F.Cu at (138.2, 88.5)
- added Q3: 2N7002, Package_TO_SOT_SMD:SOT-23, F.Cu at (138.2, 101.2)
- added R1: 10k, Resistor_SMD:R_0805_2012Metric, F.Cu at (176.0, 55.5)
- added R10: 10k, Resistor_SMD:R_0805_2012Metric, F.Cu at (165.6, 73.0)
- added R11: 10k, Resistor_SMD:R_0805_2012Metric, F.Cu at (170.1, 77.0)
- added R12: 16.2k, Resistor_SMD:R_0805_2012Metric, F.Cu at (173.1, 77.0)
- added R13: 1.00k, Resistor_SMD:R_0805_2012Metric, F.Cu at (200.6, 73.0)
- added R14: 1.00k, Resistor_SMD:R_0805_2012Metric, F.Cu at (203.6, 73.0)
- added R15: 10k, Resistor_SMD:R_0805_2012Metric, F.Cu at (197.6, 73.0)
- added R16: 10k, Resistor_SMD:R_0805_2012Metric, F.Cu at (202.1, 77.0)
- added R17: 16.2k, Resistor_SMD:R_0805_2012Metric, F.Cu at (205.1, 77.0)
- added R18: 100k, Resistor_SMD:R_0805_2012Metric, F.Cu at (136.5, 84.0)
- added R19: 100k, Resistor_SMD:R_0805_2012Metric, F.Cu at (136.5, 96.8)
- added R2: 10k, Resistor_SMD:R_0805_2012Metric, F.Cu at (210.0, 77.2)
- added R20: 100k, Resistor_SMD:R_0805_2012Metric, F.Cu at (142.3, 102.0)
- added R21: 100k, Resistor_SMD:R_0805_2012Metric, F.Cu at (142.3, 89.2)
- added R3: 100k, Resistor_SMD:R_0805_2012Metric, F.Cu at (177.8, 75.7)
- added R4: 100k, Resistor_SMD:R_0805_2012Metric, F.Cu at (207.0, 73.0)
- added R5: 1K, Resistor_SMD:R_0805_2012Metric, F.Cu at (142.2, 66.2)
- added R6: 1K, Resistor_SMD:R_0805_2012Metric, F.Cu at (142.2, 68.8)
- added R7: 1K, Resistor_SMD:R_0805_2012Metric, F.Cu at (142.2, 71.2)
- added R8: 1.00k, Resistor_SMD:R_0805_2012Metric, F.Cu at (168.6, 73.0)
- added R9: 1.00k, Resistor_SMD:R_0805_2012Metric, F.Cu at (171.6, 73.0)
- added U1: STM32G0B1CBTx, Package_QFP:LQFP-48_7x7mm_P0.5mm, F.Cu at (181.6, 64.4)
- added U2: AP63203WU, Package_TO_SOT_SMD:TSOT-23-6, F.Cu at (165.6, 63.2)
- added U3: DRV8262DDVR, Package_SO:HTSSOP-44_6.1x14mm_P0.635mm_TopEP4.14x7.01mm, F.Cu at (170.1, 84.5)
- added U4: DRV8262DDVR, Package_SO:HTSSOP-44_6.1x14mm_P0.635mm_TopEP4.14x7.01mm, F.Cu at (202.1, 84.5)
Routing:
- net GND: track 0.00 -> 228.9 mm, vias 0 -> 14
- net +3V3: track 0.00 -> 161.0 mm, vias 0 -> 7
- net /FAN2: track 0.00 -> 74.7 mm, vias 0 -> 4
- net /FAN1: track 0.00 -> 67.6 mm, vias 0 -> 4
- net +12V: track 0.00 -> 60.2 mm, vias 0 -> 100
- net /~{AB_FAULT}: track 0.00 -> 57.2 mm, vias 0 -> 2
- net /SW_LUMBAR: track 0.00 -> 53.9 mm, vias 0 -> 2
- net /SW_TILT_LIFT: track 0.00 -> 53.3 mm, vias 0 -> 2
- net /SW_BACKREST_TRACK: track 0.00 -> 52.8 mm, vias 0 -> 2
- net /~{CD_SLEEP}: track 0.00 -> 43.4 mm, vias 0 -> 2
- net /D_IN2: track 0.00 -> 38.7 mm, vias 0 -> 2
- net /D_IN1: track 0.00 -> 37.9 mm, vias 0 -> 2
- net /D_ISNS: track 0.00 -> 35.3 mm, vias 0 -> 2
- net /C_IN1: track 0.00 -> 34.6 mm, vias 0 -> 2
- net /C_ISNS: track 0.00 -> 33.0 mm, vias 0 -> 2
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- added copper zone on F.Cu, net +12V
- added copper zone on In2.Cu, net +12V
- added copper zone on F.Cu, net /Motor Driver AB/AOUT1
- added copper zone on F.Cu, net /Motor Driver AB/AOUT2
- added copper zone on F.Cu, net /Motor Driver AB/BOUT1
- added copper zone on F.Cu, net /Motor Driver AB/BOUT2
- added copper zone on F.Cu, net /Motor Driver CD/AOUT1
- added copper zone on F.Cu, net /Motor Driver CD/AOUT2
- added copper zone on F.Cu, net /Motor Driver CD/BOUT1
- added copper zone on F.Cu, net /Motor Driver CD/BOUT2
- added copper zone on In1.Cu, net GND
- added copper zone on F.Cu, net GNDPWR
- added copper zone on In1.Cu, net GNDPWR
- added copper zone on F.Cu, net Net-(J1-Pin_2)
- added copper zone on F.Cu, net Net-(Q1-D)
Other:
- board outline added: 97 x 57 mm
- copper layers 0 -> 4
